File: project/simulation/555/555/555.kicad_sch (KiCad schematic)
At the start: 7 parts, among them U1 LM555xM

Commit message: rapor hazırladım
Parts:
- C2: value 8n -> 2n
Other:
- note added: ".tran 1u 1000u 990u uic"
- note removed: ".tran 1u 10m 9.9m uic"
- moved on the sheet: C1, C2, R1, R2, R3, U1, V1
